Commit message: replaced robot model with turtlebot burger meshes

File: gym_line_follower/turtlebot3_burger.urdf (robot description, URDF)
Before this commit: robot turtlebot3_burger_min, 4 links, 3 joints
Links:
- link base_link: geometry collision cylinder length=0.12 radius=0.09; visual mesh filename=meshes/burger_base.stl scale=0.001 0.001 0.001
- link wheel_left_link: geometry collision cylinder length=0.018 radius=0.033; visual mesh filename=meshes/left_tire.stl scale=0.001 0.001 0.001
- link wheel_right_link: geometry collision cylinder length=0.018 radius=0.033; visual mesh filename=meshes/right_tire.stl scale=0.001 0.001 0.001
